Commit message: 添加基础深度相机

File: ros2_ws/src/robot_sim_demo_ros2/urdf/xbot.urdf.xacro (robot description, xacro)
@@ -2,4 +2,5 @@
 <robot name="xbot" xmlns:xacro="http://www.ros.org/wiki/xacro">
   <xacro:arg name="use_gazebo" default="false"/>
+  <xacro:arg name="enable_depth_camera" default="false"/>
   <xacro:arg name="controller_manager_config" default=""/>
   <xacro:arg name="diff_drive_controller_config" default=""/>
@@ -8,4 +9,9 @@
   <xacro:property name="wheel_radius" value="0.095"/>
   <xacro:property name="wheel_separation_half" value="0.23"/>
+  <xacro:property name="use_gazebo_arg" value="$(arg use_gazebo)"/>
+  <xacro:property name="enable_depth_camera_arg" value="$(arg enable_depth_camera)"/>
+  <xacro:property
+    name="depth_camera_enabled"
+    value="${(enable_depth_camera_arg == True or enable_depth_camera_arg == 'true' or enable_depth_camera_arg == 'True' or enable_depth_camera_arg == 1 or enable_depth_camera_arg == '1') and (use_gazebo_arg == True or use_gazebo_arg == 'true' or use_gazebo_arg == 'True' or use_gazebo_arg == 1 or use_gazebo_arg == '1')}"/>
   <link name="base_footprint"/>
   <joint name="base_footprint_to_base" type="fixed">
@@ -237,4 +243,25 @@
     <origin xyz="0 0 0" rpy="-1.5708 0 -1.5708"/>
   </joint>
+  <xacro:if value="${depth_camera_enabled}">
+    <gazebo reference="camera_link_optical">
+      <sensor name="rgbd_camera" type="rgbd_camera">
+        <always_on>true</always_on>
+        <update_rate>15</update_rate>
+        <visualize>false</visualize>
+        <topic>rgbd_camera</topic>
+        <camera>
+          <horizontal_fov>1.047</horizontal_fov>
+          <image>
+            <width>320</width>
+            <height>240</height>
+          </image>
+          <clip>
+            <near>0.1</near>
+            <far>8.0</far>
+          </clip>
+        </camera>
+      </sensor>
+    </gazebo>
+  </xacro:if>
   <gazebo reference="left_wheel">
     <mu1>10.0</mu1>
